Commit message: update readme

File: hector_quadrotor_sim/hector_quadrotor/hector_quadrotor_description/urdf/quadrotor_hokuyo_utm30lx.urdf.xacro (robot description, xacro)
@@ -8,12 +8,7 @@
     <!-- Hokuyo UTM-30LX mounted upside down below the quadrotor body -->
     <xacro:include filename="$(find hector_sensors_description)/urdf/hokuyo_utm30lx.urdf.xacro" />
-    <!-- CUSTON XACRO HOKUYO MAX AND MIN ANGLE - OBS: FRONT ALING WITH 0 DEGREE LASER HOKUYO-->
-    <xacro:hokuyo_utm30lx name="laser0" parent= "base_link" ros_topic="scan" update_rate="40" ray_count="1081" min_angle="0" max_angle="360">
+    <xacro:hokuyo_utm30lx name="laser0" parent="base_link" ros_topic="scan" update_rate="40" ray_count="1081" min_angle="-135" max_angle="135">
       <origin xyz="0.0 0.0 -0.097" rpy="${M_PI} 0 0"/>
     </xacro:hokuyo_utm30lx>
-    <!-- ORIGINAL XACRO HOKUYO MAX AND MIN ANGLE -->
-    <!-- <xacro:hokuyo_utm30lx name="laser0" parent="base_link" ros_topic="scan" update_rate="40" ray_count="1081" min_angle="-135" max_angle="135">
-      <origin xyz="0.0 0.0 -0.097" rpy="${M_PI} 0 0"/>
-    </xacro:hokuyo_utm30lx> -->
     <!-- Forward facing camera -->
     <xacro:include filename="$(find hector_sensors_description)/urdf/generic_camera.urdf.xacro" />
